Commit message: added T265, stable version

File: pippino_description/src/description/_d455.urdf.xacro (robot description, xacro)
@@ -11,5 +11,5 @@
   <xacro:include filename="$(find pippino_description)/src/description/_usb_plug.urdf.xacro" />
   <xacro:macro name="sensor_d455" params="parent *origin name:=camera use_nominal_extrinsics:=false">
-    <xacro:arg name="add_plug" default="false" />
+    <xacro:arg name="add_plug" default="true" />
     <xacro:property name="M_PI" value="3.1415926535897931" />
     <!-- The following values are approximate, and the camera node
@@ -51,9 +51,9 @@
       <visual>
         <!-- the mesh origin is at front plate in between the two infrared camera axes -->
-        <!-- <origin xyz="${d455_zero_depth_to_glass-d455_cam_depth/2} ${-d455_cam_depth_py} 0" rpy="0 0 0"/> -->
-        <origin xyz="${d455_zero_depth_to_glass + d455_glass_to_front} ${-d455_cam_depth_py} 0" rpy="${M_PI/2} 0 ${M_PI/2}"/>
+        <origin xyz="${d455_zero_depth_to_glass-d455_cam_depth/2} ${-d455_cam_depth_py} 0" rpy="0 0 0"/>
+        <!-- <origin xyz="${d455_zero_depth_to_glass + d455_glass_to_front} ${-d455_cam_depth_py} 0" rpy="${M_PI/2} 0 ${M_PI/2}"/> -->
         <geometry>
-          <!-- <box size="${d455_cam_depth} ${d455_cam_width} ${d455_cam_height}"/> -->
-	        <mesh filename="$(find pippino_description)/meshes/d455.stl" scale="0.001 0.001 0.001" />
+          <box size="${d455_cam_depth} ${d455_cam_width} ${d455_cam_height}"/>
+	        <!-- <mesh filename="$(find pippino_description)/meshes/d455.stl" scale="0.001 0.001 0.001" /> -->
         </geometry>
         <material name="aluminum"/>

File: pippino_description/src/description/_usb_plug.urdf.xacro (robot description, xacro)
@@ -19,6 +19,6 @@
         <origin xyz="0. -0.022425 0." rpy="0 0 ${M_PI/2}"/>
         <geometry>
-          <!--box size="0.044850 0.008 0.0185" /-->
-          <mesh filename="$(find pippino_description)/meshes/plug.stl" />
+          <box size="0.044850 0.008 0.0185" />
+          <!-- <mesh filename="$(find pippino_description)/meshes/plug.stl" /> -->
         </geometry>
         <material name="plastic"/>
@@ -27,6 +27,6 @@
         <origin xyz="0. -0.022425 0." rpy="0 0 ${M_PI/2}"/>
         <geometry>
-          <!--box size="0.044850 0.008 0.0185" /-->
-          <mesh filename="$(find pippino_description)/meshes/plug_collision.stl" />
+          <box size="0.044850 0.008 0.0185" />
+          <!-- <mesh filename="$(find pippino_description)/meshes/plug_collision.stl" /> -->
         </geometry>
       </collision>

File: pippino_description/src/description/pippino.urdf (robot description, URDF)
Before this commit: robot pippino, 6 links, 5 joints
Links:
- removed link camera_link
- added link T265_pose_frame; visual box size=0.03 0.12 0.03
- added link aruco_marker; visual box size=0.175 0.175 0.002
- added link body_link
- added link charging_position; visual cylinder length=0.005 radius=0.01
- added link charging_position_rough; visual cylinder length=0.005 radius=0.01
- added link charging_station; visual box size=0.16 0.4 0.04
- added link charging_station_connector; visual cylinder length=0.006 radius=0.01
- added link power_connector; visual cylinder length=0.006 radius=0.01
- added link power_probe; visual cylinder length=0.142 radius=0.004
Joints:
- removed joint camera_joint
- added joint T265_pose_joint: type fixed, parent body_link, child T265_pose_frame, origin xyz=0.053 0.0 0.225 rpy=0.0 0.0 0.0
- added joint aruco_marker_joint: type floating, parent D455_color_optical_frame, child aruco_marker, origin xyz=0 0 0.005 rpy=0 0 0
- added joint body_joint: type fixed, parent base_link, child body_link, origin xyz=-0.08 0 0 rpy=0 0 0
- added joint charging_position_joint: type fixed, parent aruco_marker, child charging_position, origin xyz=0 -0.214 0.224 rpy=-${pi/2} ${pi/2} 0
- added joint charging_position_joint_rough: type fixed, parent charging_position, child charging_position_rough, origin xyz=-0.1 0 0 rpy=0 0 0
- added joint charging_station_connector_joint: type fixed, parent aruco_marker, child charging_station_connector, origin xyz=0.027 -0.16 0.003 rpy=0 0 0
- added joint charging_station_joint: type fixed, parent aruco_marker, child charging_station, origin xyz=0.0 -0.008 -0.04 rpy=0 0 0
- added joint power_connector_joint: type fixed, parent power_probe, child power_connector, origin xyz=0.142 0.0 0.0 rpy=0 0 0
- added joint power_probe_joint: type revolute, parent body_link, child power_probe, origin xyz=${base_length/2 - 0.01} -0.025 0.05 rpy=${pi} 0 ${pi/2}, axis 0 0 1, limit lower=0.0 upper=${pi/2} effort=10 velocity=0.5
- joint back_wheel_joint: parent base_link -> body_link
- joint base_footprint_joint: parent base_link -> body_link
- joint circuits_joint: parent base_link -> body_link
- joint laser_joint: parent base_link -> body_link
