Commit message: working, ok velocity and settings

File: pippino_description/src/description/pippino.urdf (robot description, URDF)
Before this commit: robot pippino, 5 links, 4 joints
Joints:
- joint camera_joint: origin xyz=-0.10 0.13 0.22 rpy=0.0 0.0 0.0 -> xyz=-0.10 0.13 0.21 rpy=0.0 0.0 0.0

Commit message: work

File: pippino_description/src/description/pippino.urdf (robot description, URDF)
Before this commit: robot pippino, 5 links, 4 joints
Joints:
- joint camera_joint: origin xyz=-0.10 0.13 0.21 rpy=0.0 0.0 0.0 -> xyz=-0.066 0.05 0.21 rpy=0.0 0.0 0.0
- joint laser_joint: origin xyz=-0.155 0.0 0.18 rpy=0 0 3.14159265 -> xyz=-0.155 0.0 0.18 rpy=0 0 3.1

Commit message: moved to humble. working status. using galactic for realsense due to bug in setting params for t265

File: pippino_description/src/description/pippino.urdf (robot description, URDF)
Before this commit: robot pippino, 14 links, 13 joints
Links:
- removed link aruco_marker
- removed link charging_position
- removed link charging_position_rough
- removed link charging_station
- removed link charging_station_connector
Joints:
- removed joint aruco_marker_joint
- removed joint charging_position_joint
- removed joint charging_position_joint_rough
- removed joint charging_station_connector_joint
- removed joint charging_station_joint
- joint laser_joint: origin xyz=-0.067 0.0 0.134 rpy=0 0 3.1 -> xyz=-0.067 0.0 0.134 rpy=0 0 3.142

Commit message: almost working pippino 2.3

File: pippino_description/src/description/pippino.urdf (robot description, URDF)
Before this commit: robot pippino, 9 links, 8 joints
Links:
- removed link circuits
Joints:
- removed joint circuits_joint
- joint laser_joint: origin xyz=-0.067 0.0 0.134 rpy=0 0 3.142 -> xyz=0.0 0.0 0.235 rpy=0 0 1.57
